Commit message: 4th-week init

File: urdf/robot.urdf (robot description, URDF)
Before this commit: robot gazebo_one_joint, 2 links, 1 joints
Links:
- removed link base_link
- removed link second_link
- added link chassis, mass 15.0; collision box size=.4 .2 .1; collision sphere radius=0.05
- added link left_wheel, mass 5; collision cylinder length=0.05 radius=0.1; visual cylinder length=0.05 radius=0.1
- added link right_wheel, mass 5; collision cylinder length=0.05 radius=0.1; visual cylinder length=0.05 radius=0.1
Joints:
- removed joint base_to_second_joint
- added joint left_wheel_hinge: type continuous, parent chassis, child left_wheel, origin xyz=0 0.15 0 rpy=0 0 0, axis 0 1 0, limit effort=10000 velocity=1000
- added joint right_wheel_hinge: type continuous, parent chassis, child right_wheel, origin xyz=0 -0.15 0 rpy=0 0 0, axis 0 1 0, limit effort=10000 velocity=1000
